File: Mark-3.kicad_pcb (KiCad board)
At the start: 2 copper layers, 121.3 x 132.8 mm, 310 parts, among them J1 Conn_01x02_Pin, J10 Conn_01x03_Pin, J11 Conn_01x03_Pin, J12 Conn_01x03_Pin, J13 Conn_01x03_Pin, J14 Conn_01x03_Pin, J15 Conn_01x03_Pin, J2 TYPE-C-31-M-12, J3 TYPE-C-31-M-12, J4 Conn_01x03_Pin, J5 Conn_01x03_Pin, J6 Conn_01x03_Pin, J7 Conn_01x03_Pin, J8 Conn_01x03_Pin, J9 Conn_01x03_Pin, Q1 HSBA4052, Q2 HSBA4052, Q3 FS8205A, Q4 FS8205A, Q5 FS8205A, Q6 FS8205A, Q7 FS8205A, Q8 FS8205A, SW1 KMR221GLFS, SW2 KMR221GLFS, U1 USBLC6-2SC6, U10 INA180A2, U11 INA180A2, U2 DW01A, U3 DW01A, U4 DW01A, U5 DW01A, U6 DW01A, U7 DW01A, U8 INA180A2, U9 INA180A2, Y1 16MHz, Y2 16MHz

Commit message: rev0 ready
Parts:
- removed TP10, TP11, TP12: TestPoint, TestPoint:TestPoint_Pad_D1.0mm
- added G***: LOGO, LOGO, B.Cu at (165.5, 144.5)
- added G***: LOGO, LOGO, B.Cu at (165.3, 48.5)
- added G***: LOGO, LOGO, B.Cu at (170.7, 96.3)
- added TP8: TestPoint, TestPoint:TestPoint_Pad_D1.0mm, F.Cu at (128.9, 97.7)
- added kibuzzard-68E68F97: G***, kibuzzard-68E68F97, F.Cu at (104.8, 134.8)
- moved TP8 199.6 mm to (256.9, 190.6)
- moved R46 155.8 mm to (123.4, 105.9), turned to 180 degrees
- moved R45 155.7 mm to (123.4, 106.6)
- moved R37 153.4 mm to (116.5, 90.7), turned to 180 degrees
- moved R15 145.7 mm to (105.1, 151.3)
- moved C54 144.6 mm to (127.5, 140.8), turned to -90 degrees
- moved R32 143.6 mm to (105.4, 104.1), turned to -45 degrees
- moved R14 142.3 mm to (99.6, 152.3), turned to 180 degrees
- moved R33 139.7 mm to (104.8, 104.7), turned to -45 degrees
- moved R9 138.3 mm to (99.2, 132.2), turned to -90 degrees
- moved R34 137.4 mm to (102.5, 105.3), turned to 180 degrees
- moved C6 136.5 mm to (105.1, 152.3)
- moved R36 135.6 mm to (99.2, 135.3), turned to -90 degrees
- moved R40 133.5 mm to (99.2, 133.9), turned to 90 degrees
- moved Y2 131.5 mm to (116.5, 88.2), turned to 90 degrees
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Connections:
- C48 pad 2: Net-(Q2-D) -> Net-(DD6-PH)
- DD5 pad 1: Leg1_servo3 -> Net-(DD5-GPIO4)
- DD5 pad 11: Leg4_servo2 -> 6V_1_EN
- DD5 pad 12: Leg4_servo3 -> LVL1
- DD5 pad 13: LVL1 -> LVL2
- DD5 pad 14: LVL2 -> LVL3
- DD5 pad 16: LVL3 -> LVL4
- DD5 pad 17: LVL4 -> LVL5
- DD5 pad 18: LVL5 -> LVL6
- DD5 pad 19: LVL6 -> LVL7
- DD5 pad 2: Leg2_servo1 -> Net-(DD5-GPIO5)
- DD5 pad 20: LVL7 -> LVL8
- DD5 pad 21: LVL8 -> Leg4_servo3
- DD5 pad 22: LED1 -> Leg4_servo2
- DD5 pad 23: LED2 -> Leg4_servo1
- DD5 pad 25: Net-(DD5-GPIO24) -> Leg3_servo3
- DD5 pad 26: Net-(DD5-GPIO25) -> Leg3_servo2
- DD5 pad 27: Net-(DD5-GPIO26) -> Leg3_servo1
- DD5 pad 28: SPI_MOSI -> Leg2_servo3
- DD5 pad 3: Leg2_servo2 -> Net-(DD5-GPIO6)
- DD5 pad 33: Net-(DD5-SWCLK) -> unconnected-(DD5-SWCLK-Pad33)
- DD5 pad 34: Net-(DD5-SWDIO) -> unconnected-(DD5-SWDIO-Pad34)
- DD5 pad 36: SPI_MISO -> Leg2_servo2
- DD5 pad 37: SPI_SCK -> Leg2_servo1
- DD5 pad 38: NRF_CS -> Leg1_servo3
- DD5 pad 39: NRF_CE -> Leg1_servo2
- DD5 pad 4: Leg2_servo3 -> Net-(DD5-GPIO7)
- DD5 pad 40: NRF_IRQ -> Leg1_servo1
- DD5 pad 45: 6V_1_EN -> SPI_MISO
- DD5 pad 46: 6V_2_EN -> NRF_CS
- DD5 pad 47: 6V_3_EN -> SPI_SCK
- DD5 pad 48: 6V_4_EN -> SPI_MOSI
- DD5 pad 49: BAT_ADC -> NRF_CE
- DD5 pad 52: 6V_1_current -> NRF_IRQ
- DD5 pad 53: 6V_2_current -> 6V_1_current
- DD5 pad 54: 6V_3_current -> 6V_2_current
- DD5 pad 55: 6V_4_current -> 6V_3_current
- DD5 pad 56: Net-(DD5-GPIO45_ADC5) -> 6V_4_current
- DD5 pad 57: Net-(DD5-GPIO46_ADC6) -> BAT_ADC
- DD5 pad 58: Net-(DD5-GPIO47_ADC7) -> unconnected-(DD5-GPIO47_ADC7-Pad58)
- DD5 pad 6: Leg3_servo1 -> Net-(DD5-GPIO8)
- DD5 pad 7: Leg3_servo2 -> 6V_4_EN
- DD5 pad 77: Net-(DD5-GPIO0) -> LED1
- DD5 pad 78: Net-(DD5-GPIO1) -> LED2
- DD5 pad 79: Leg1_servo1 -> Net-(DD5-GPIO2)
- DD5 pad 8: Leg3_servo3 -> 6V_3_EN
- DD5 pad 80: Leg1_servo2 -> Net-(DD5-GPIO3)
- DD5 pad 9: Leg4_servo1 -> 6V_2_EN
- DD6 pad 20: unconnected-(DD6-PH-Pad20) -> Net-(DD6-PH)
- L6 pad 1: Net-(Q2-D) -> Net-(DD6-PH)
- Q1 pad 1: Net-(Q2-D) -> Net-(DD6-PH)
- Q1 pad 2: Net-(Q2-D) -> Net-(DD6-PH)
- Q1 pad 3: Net-(Q2-D) -> Net-(DD6-PH)
- Q2 pad 5: Net-(Q2-D) -> Net-(DD6-PH)
- TP3 pad 1: Net-(DD5-GPIO0) -> Net-(DD5-GPIO2)
- TP4 pad 1: Net-(DD5-GPIO1) -> Net-(DD5-GPIO3)
- TP5 pad 1: Net-(DD5-GPIO24) -> Net-(DD5-GPIO4)
- TP6 pad 1: Net-(DD5-GPIO25) -> Net-(DD5-GPIO5)
- TP7 pad 1: Net-(DD5-GPIO26) -> Net-(DD5-GPIO6)
- TP9 pad 1: Net-(DD5-GPIO46_ADC6) -> Net-(DD5-GPIO8)
Routing:
- net VBAT: track 0.00 -> 336.7 mm, vias 0 -> 45
- net 3.3V: track 0.00 -> 201.8 mm, vias 0 -> 35
- net 6V_1_EN: track 0.00 -> 103.3 mm, vias 0 -> 2
- net 6V_1_current: track 0.00 -> 99.7 mm, vias 0 -> 2
- net 6V_2_EN: track 0.00 -> 91.2 mm, vias 0 -> 2
- net 6V_2_current: track 0.00 -> 88.8 mm, vias 0 -> 2
- net 6V_3_EN: track 0.00 -> 79.5 mm, vias 0 -> 2
- net Leg1_servo3: track 0.00 -> 77.4 mm
- net 6V_3_current: track 0.00 -> 76.1 mm, vias 0 -> 2
- net Leg1_servo2: track 0.00 -> 74.9 mm
- net Leg2_servo3: track 0.00 -> 73.0 mm
- net Leg1_servo1: track 0.00 -> 72.6 mm
- net Net-(DD5-RUN): track 0.00 -> 68.8 mm, vias 0 -> 2
- net 6V_4_EN: track 0.00 -> 66.8 mm, vias 0 -> 2
- net Net-(DD6-VFB): track 0.00 -> 64.1 mm, vias 0 -> 4
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- added copper zone on B.Cu, net 3.3V
- added copper zone on F.Cu, net 3.3V
- added copper zone on B.Cu, net 6V_1
- added copper zone on F.Cu, net 6V_1
- added copper zone on B.Cu, net 6V_2
- added copper zone on F.Cu, net 6V_2
- added copper zone on B.Cu, net 6V_3
- added copper zone on F.Cu, net 6V_3
- added copper zone on B.Cu, net 6V_4
- added copper zone on F.Cu, net 6V_4
- added copper zone on B.Cu, net Earth
- added copper zone on F.Cu, net Earth
- added copper zone on F.Cu, net Net-(BT1--)
- added copper zone on F.Cu, net Net-(BT2--)
- added copper zone on F.Cu, net Net-(BT3--)
- added copper zone on F.Cu, net Net-(BT4--)
- added copper zone on F.Cu, net Net-(BT5--)
- added copper zone on F.Cu, net Net-(BT6--)
- added copper zone on F.Cu, net Net-(DD10-SW_1)
- added copper zone on F.Cu, net Net-(DD10-VOUT_1)
- added copper zone on F.Cu, net Net-(DD11-SW_1)
- added copper zone on F.Cu, net Net-(DD11-VOUT_1)
- added copper zone on F.Cu, net Net-(DD5-ADC_AVDD)
- added copper zone on F.Cu, net Net-(DD5-DVDD_1)
- added copper zone on F.Cu, net Net-(DD5-VREG_LX)
- added copper zone on F.Cu, net Net-(DD6-PH)
- added copper zone on F.Cu, net Net-(DD6-SRP)
- added copper zone on F.Cu, net Net-(DD8-SW_1)
- added copper zone on F.Cu, net Net-(DD8-VOUT_1)
- added copper zone on F.Cu, net Net-(DD9-SW_1)
- added copper zone on F.Cu, net Net-(DD9-VOUT_1)
- added copper zone on B.Cu, net VBAT
- added copper zone on F.Cu, net VBAT
- added copper zone on B.Cu, net VUSB
- added copper zone on F.Cu, net VUSB
Other:
- board size 121.3 x 132.8 mm -> 125.2 x 132.8 mm
- board text added: "LEG 1"
- board text added: "LEG 2"
- board text added: "LEG 3"
- board text added: "LEG 4"
- board text added: "PWR"
- board text added: "USB"
- board text added: "by @madjogger"
